Commit message: URDF Model

File: robot1_description/robots/robot1.urdf (robot description, URDF)
Before this commit: robot test_robot, 3 links, 2 joints
Links:
- removed link link1
- removed link link2
- removed link link3
- added link servo_right_left
- added link servo_up_down
- added link webcam1
- added link world
Joints:
- removed joint joint1
- removed joint joint2
- added joint join1_base_to_head: type continuous, parent world, child servo_right_left, origin xyz=0 0 0 rpy=0 0 0
- added joint join1_head_to_camera: type continuous, parent world, child servo_right_left, origin xyz=0 0 0 rpy=0 0 0
- added joint single_rrbot_fixed: type fixed, parent world, child servo_right_left, origin xyz=0 0 0 rpy=0 0 0

Commit message: Robot1.urdf las version

File: robot1_description/robots/robot1.urdf (robot description, URDF)
Before this commit: robot robot1_webcam, 4 links, 3 joints
Links:
- added link electronic_box; visual box size=0.175 .125 0.045
- link servo_right_left: geometry visual box size=0.055 0.020 0.045
- link servo_up_down: geometry visual box size=0.04 0.020 0.055
- link webcam1: geometry visual sphere radius=0.03
Joints:
- removed joint join1_base_to_head
- removed joint join1_head_to_camera
- added joint join1_box_to_servo1: type fixed, parent electronic_box, child servo_right_left, origin xyz=0 -0.05 0 rpy=0 0 0
- added joint join2_base_to_head: type revolute, parent servo_right_left, child servo_up_down, origin xyz=0 0 0.045 rpy=0 0 0, axis 0 0 1, limit lower=-1.57 upper=1.57 effort=100.0 velocity=0.5
- added joint join3_head_to_camera: type revolute, parent servo_up_down, child webcam1, origin xyz=0.01 0.00 0.01 rpy=0 0 0, axis 1 0 0, limit lower=-1.57 upper=1.57 effort=10.0 velocity=0.5
- joint single_rrbot_fixed: child servo_right_left -> electronic_box

Commit message: Updated Lense

File: robot1_description/robots/robot1.urdf (robot description, URDF)
Before this commit: robot robot1, 5 links, 4 joints
Links:
- added link lense; visual cylinder length=0.005 radius=0.017
Joints:
- added joint webcam1_to_lense: type fixed, parent webcam1, child lense, origin xyz=0 0 0 rpy=0 0 0
